File: Embedded_headstart_board.kicad_pcb (KiCad board)
At the start: 2 copper layers, 100 x 100 mm, 145 parts, among them J101 86093488324755V1LF, J102 Jumper, J103 BMP280, J104 Jumper, J105 MPU-6500, J106 ADDR Sel, J107 BMP280, J108 MPU-6500, U101 DHT11, U102 SN74CB3Q3245PWR, U103 TCA9535PWR_C130204, U104 TCA9535PWR_C130204, U105 TCA9535PWR_C130204, U107 9001-17481C00A_C5173377, U108 SN74CB3Q3245PWR, U109 AMS1117, U202 74HC595D, U301 74HC595D, U401 74HC595D, U501 74HC595D

Commit message: MORE STUFF
Parts:
- removed D105, D109, D125, D129: Red, Custom_footprints:Multi_diode
- removed R107, R111, R136, R139: 1kΩ, PCM_JLCPCB:R_0603
- D123, D124: footprint Custom_footprints:Multi_diode -> PCM_JLCPCB:D_0603
- moved C101 134.7 mm to (324.2, 71.8)
- moved C107 124.5 mm to (330.8, 114.5)
- moved C108 124.5 mm to (330.8, 116.7)
- moved R128 124.5 mm to (319.7, 116.7)
- moved R132 124.5 mm to (323.4, 103.2)
- moved R133 124.5 mm to (323.4, 105.5)
- moved R137 124.5 mm to (323.4, 114.5)
- moved R138 124.5 mm to (323.4, 116.7)
- moved U102 110.6 mm to (354.2, 110.4), turned to -90 degrees
- moved R127 109.1 mm to (332.6, 126.2), turned to 90 degrees
- moved R131 109.1 mm to (334.3, 126.2), turned to 90 degrees
- moved U103 108.5 mm to (369.8, 111.4), turned to -90 degrees
- moved R118 106.6 mm to (335.5, 70.1)
- moved R109 106.6 mm to (331.9, 72.3)
- moved R110 106.6 mm to (331.9, 74.6)
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Connections:
- U103 pad 4: Net-(U103-P00) -> unconnected-(U103-P00-Pad4)
- U103 pad 7: Net-(U103-P03) -> unconnected-(U103-P03-Pad7)
- U104 pad 4: Net-(U104-P00) -> unconnected-(U104-P00-Pad4)
- U104 pad 7: Net-(U104-P03) -> unconnected-(U104-P03-Pad7)
Other:
- board text added: "Bus Switch #1"
- board text added: "GPIO Expander"

Commit message: V1.0
Parts:
- removed J101: 86093488324755V1LF, Connector_DIN:DIN41612_C2_3x16_Female_Vertical_THT
- added G***: LOGO, Custom_footprints:Repo_QR, F.Cu at (291.8, 101.3)
- added konar1: LOGO, Custom:konar, F.Cu at (36.7, 44.6)
- moved D127 312.0 mm to (77.1, 117.4)
- moved D111 312.0 mm to (33.9, 109.4)
- moved D121 312.0 mm to (70.6, 122.2), turned to 180 degrees
- moved S106 312.0 mm to (75.3, 123.8)
- moved S107 312.0 mm to (75.3, 132.4)
- moved D122 312.0 mm to (70.4, 130.7)
- moved R134 312.0 mm to (70.6, 124.0)
- moved R135 312.0 mm to (70.4, 132.5)
- moved R140 312.0 mm to (70.6, 125.6)
- moved R142 312.0 mm to (70.4, 134.1)
- moved U102 312.0 mm to (42.3, 117.1)
- moved U103 312.0 mm to (57.9, 118.1)
- moved D112 312.0 mm to (48.8, 129.1)
- moved D126 312.0 mm to (77.1, 108.4)
- moved D101 311.9 mm to (42.2, 129.1)
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Connections:
- net /Chainbus.CS renamed /CSB
- net /Chainbus.MISO renamed /ADD
- J102 pad 1: Net-(J102-Pin_1) -> /Chainbus.SDA
- J102 pad 2: /Chainbus.SDA -> Net-(J102-Pin_2)
- J104 pad 1: Net-(J104-Pin_1) -> /Chainbus.SCL
- J104 pad 2: /Chainbus.SCL -> Net-(J104-Pin_2)
- J105 pad 10: /ECL -> /Altmode3
- J105 pad 6: /ECL -> /Altmode6
- J105 pad 8: /ECL -> /Altmode1
- J105 pad 9: /Chainbus.RX -> /Altmode2
- J108 pad 10: /ECL -> /Altmode3
- J108 pad 6: /ECL -> /Altmode6
- J108 pad 8: /ECL -> /Altmode1
- J108 pad 9: /Chainbus.RX -> /Altmode2
- R101 pad 1: /ECL -> /Chainbus_addr4
- R102 pad 1: /ECL -> /Chainbus_addr0
- R104 pad 1: /ECL -> /Chainbus_addr3
- R105 pad 1: Net-(S103-A) -> /E1_P15
- R106 pad 1: Net-(S102-A) -> /E1_P14
- R108 pad 1: Net-(S104-A) -> /E3_P15
- R109 pad 1: Net-(U104-P01) -> /E1_P16
- R110 pad 1: Net-(U104-P02) -> /E1_P17
- R112 pad 2: Net-(S105-A) -> /E3_P14
- R113 pad 1: Net-(S104-A) -> /E3_P15
- R114 pad 1: Net-(S105-A) -> /E3_P14
- R117 pad 2: /ECL -> /Chainbus.RX
- R118 pad 2: /ECL -> /Chainbus.TX
- R120 pad 1: Net-(U105-P00) -> /E3_P16
- R121 pad 1: Net-(U105-P01) -> /E3_P17
- R125 pad 2: /ECL -> /Chainbus_addr5
- R126 pad 1: /ECL -> /Chainbus_addr5
- R128 pad 2: /ECL -> /Chainbus_addr2
- R129 pad 1: Net-(S103-A) -> /E1_P15
- R130 pad 2: Net-(S102-A) -> /E1_P14
- R134 pad 1: Net-(S106-A) -> /E2_P15
- R135 pad 2: Net-(S107-A) -> /E2_P14
- R137 pad 1: Net-(U103-P01) -> /E2_P16
- R138 pad 1: Net-(U103-P02) -> /E2_P17
- R140 pad 1: Net-(S106-A) -> /E2_P15
- R141 pad 2: /ECL -> /Chainbus_addr7
- R142 pad 1: Net-(S107-A) -> /E2_P14
- R143 pad 2: /ECL -> /Altmode1
- R144 pad 1: /ECL -> /Altmode3
- S101 pad 1: /ECL -> /Chainbus_addr3
- S102 pad 1: Net-(S102-A) -> /E1_P14
- S103 pad 1: Net-(S103-A) -> /E1_P15
- S104 pad 1: Net-(S104-A) -> /E3_P15
- S105 pad 1: Net-(S105-A) -> /E3_P14
- S106 pad 1: Net-(S106-A) -> /E2_P15
- S107 pad 1: Net-(S107-A) -> /E2_P14
- U101 pad 2: /ECL -> /Chainbus.RX
- U102 pad 19: /ECL -> /Chainbus_addr2
- U102 pad 4: /ECL -> /Chainbus_addr1
- U103 pad 17: unconnected-(U103-P14-Pad17) -> /E2_P14
- U103 pad 18: unconnected-(U103-P15-Pad18) -> /E2_P15
- U103 pad 19: unconnected-(U103-P16-Pad19) -> /E2_P16
- U103 pad 20: unconnected-(U103-P17-Pad20) -> /E2_P17
- U103 pad 5: Net-(U103-P01) -> unconnected-(U103-P01-Pad5)
- U103 pad 6: Net-(U103-P02) -> unconnected-(U103-P02-Pad6)
- U103 pad 8: Net-(S106-A) -> unconnected-(U103-P04-Pad8)
- U103 pad 9: Net-(S107-A) -> unconnected-(U103-P05-Pad9)
- U104 pad 1: /ECL -> /Chainbus.TX
- U104 pad 17: unconnected-(U104-P14-Pad17) -> /E1_P14
- U104 pad 18: unconnected-(U104-P15-Pad18) -> /E1_P15
- U104 pad 19: unconnected-(U104-P16-Pad19) -> /E1_P16
- U104 pad 20: unconnected-(U104-P17-Pad20) -> /E1_P17
- U104 pad 22: Net-(J104-Pin_1) -> Net-(J104-Pin_2)
- U104 pad 23: Net-(J102-Pin_1) -> Net-(J102-Pin_2)
- U104 pad 5: Net-(U104-P01) -> unconnected-(U104-P01-Pad5)
- U104 pad 6: Net-(U104-P02) -> unconnected-(U104-P02-Pad6)
- U104 pad 8: Net-(S103-A) -> unconnected-(U104-P04-Pad8)
- U104 pad 9: Net-(S102-A) -> unconnected-(U104-P05-Pad9)
- U105 pad 17: unconnected-(U105-P14-Pad17) -> /E3_P14
- U105 pad 18: unconnected-(U105-P15-Pad18) -> /E3_P15
- U105 pad 19: unconnected-(U105-P16-Pad19) -> /E3_P16
- U105 pad 20: unconnected-(U105-P17-Pad20) -> /E3_P17
- U105 pad 4: Net-(U105-P00) -> unconnected-(U105-P00-Pad4)
- U105 pad 5: Net-(U105-P01) -> unconnected-(U105-P01-Pad5)
- U105 pad 6: Net-(S104-A) -> unconnected-(U105-P02-Pad6)
- U105 pad 7: Net-(S105-A) -> unconnected-(U105-P03-Pad7)
- U107 pad A5: BRD_VIN -> unconnected-(U107-PadA5)
- U107 pad A6: BRD_VIN -> unconnected-(U107-PadA6)
- U107 pad A7: BRD_VIN -> unconnected-(U107-PadA7)
- U107 pad A8: BRD_VIN -> unconnected-(U107-PadA8)
- U108 pad 19: /ECL -> /Chainbus_addr7
- U108 pad 4: /ECL -> /Chainbus_addr6
- U202 pad 11: /ECL -> /Altmode12
- U202 pad 12: /ECL -> /Altmode13
- U202 pad 13: /ECL -> /Altmode14
- U202 pad 14: /ECL -> /Altmode15
- U301 pad 11: /ECL -> /Altmode12
- U301 pad 12: /ECL -> /Altmode13
- U301 pad 13: /ECL -> /Altmode14
- U401 pad 11: /ECL -> /Altmode12
- U401 pad 12: /ECL -> /Altmode13
- U401 pad 13: /ECL -> /Altmode14
- U501 pad 11: /ECL -> /Altmode12
- U501 pad 12: /ECL -> /Altmode13
- U501 pad 13: /ECL -> /Altmode14
Routing:
- net +3V3: track 5.50 -> 742.7 mm, vias 0 -> 24
- net /Altmode14: track 0.00 -> 262.1 mm, vias 0 -> 4
- net /Altmode13: track 0.00 -> 256.3 mm, vias 0 -> 4
- net /Altmode12: track 0.00 -> 249.8 mm, vias 0 -> 4
- net /Chainbus.SCK: track 0.00 -> 246.9 mm
- net /Chainbus.MOSI: track 0.00 -> 241.2 mm, vias 0 -> 1
- net /ADD: track 0.00 -> 233.0 mm
- net /Altmode15: track 0.00 -> 216.9 mm
- net /CSB: track 0.00 -> 197.4 mm, vias 0 -> 1
- net /Altmode6: track 0.00 -> 158.5 mm
- net /Altmode1: track 0.00 -> 157.3 mm
- net /Altmode2: track 0.00 -> 139.7 mm
- net /Altmode3: track 0.00 -> 135.5 mm
- net /Chainbus.RX: track 0.00 -> 135.2 mm, vias 0 -> 1
- net /Chainbus.SDA: track 0.00 -> 129.2 mm, vias 0 -> 4
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- added copper zone on B.Cu, net +3V3
- added copper zone on F.Cu, net +3V3
- added copper zone on B.Cu, net GND
- added copper zone on F.Cu, net GND
Other:
- board size 100 x 100 mm -> 120 x 170 mm
- board text added: "DIN: PC3 OE#: PC2 SHCP: PC0 STCP: PC1"
- board text added: "Data: PC11"
- board text added: "I think you should turn me around..."
- board text added: "I2C SDA: PB11 SCL: PB10"
- board text added: "IT PC10"
- board text added: "LED Both Types"
- board text added: "Made by Wojtek Szafrański Version 1.0"
- board text added: "Manual Bus Switch"
- board text added: "NC"
- board text added: "OE# (Act. Low): PA5"
- board text added: "OE# (Act. Low): PC8"
- board text added: "P14"
- board text added: "P15"
- board text added: "P16"
- board text added: "P17"
- board text added: "PA6"
- board text added: "PA7 LED Active High"
- board text added: "PB5 LED Active High"
- board text added: "PC6"
- board text added: "PC7"
- board text added: "PC9 Button Active High"
- board text added: "Readme QR"
- board text added: "SCL: PB3 SDA: PC12 EDA: NC ECL: PB15 ADD: PB4 INT: PA8 NCS: PA9 FSYNC: PA10"
- board text removed: "DIN: PXX OE#: PXX SHCP: PXX STCP: PXX"
- board text removed: "DON'T PUT ANYTHING HERE"
- board text removed: "Data: PXX"
- board text removed: "OE# (Act. Low): PXX"
- board text removed: "PXX"
- board text removed: "PXX Button Active High"
- board text removed: "PXX LED Active High"
- board text removed: "PXX Two types"
- board text removed: "SCL: PB3 SDA: PC12 EDA: NC ECL: PXX ADD: PB4 INT: PXX NCS: PC11 FSYNC: PXX"
