File: Embedded_headstart_board.kicad_sch (KiCad schematic)
At the start: 101 parts, among them J101 86093488324755V1LF, J102 Jumper, J103 BMP280, J104 Jumper, J105 MPU-6500, J106 ADDR Sel, J107 BMP280, J108 MPU-6500, U101 DHT11, U102 SN74CB3Q3245PWR, U103 TCA9535PWR_C130204, U104 TCA9535PWR_C130204, U105 TCA9535PWR_C130204, U107 9001-17481C00A_C5173377, U108 SN74CB3Q3245PWR, U109 AMS1117

Commit message: MORE STUFF
Parts:
- removed D105, D109, D125, D129: Red, Custom_footprints:Multi_diode, symbol PCM_JLCPCB-Diodes:LED,0603,Red
- removed R107, R111, R136, R139: 1kΩ, PCM_JLCPCB:R_0603, symbol PCM_JLCPCB-Resistors:0603,1kΩ
- D123, D124: footprint Custom_footprints:Multi_diode -> PCM_JLCPCB:D_0603
Connections:
- no-connect marks 53 -> 55
Other:
- moved on the sheet: D126

Commit message: V1.0
Parts:
- removed J101: 86093488324755V1LF, Connector_DIN:DIN41612_C2_3x16_Female_Vertical_THT, symbol 86093488324755V1LF:86093488324755V1LF
Connections:
- net Altmode1: now also J105.8 (Pin_8), J108.8 (Pin_8), R143.2
- net Altmode2: now also J105.9 (Pin_9), J108.9 (Pin_9)
- net Altmode3: now also J105.10 (Pin_10), J108.10 (Pin_10), R144.1
- net Altmode6: now also J105.6 (Pin_6), J108.6 (Pin_6)
- net BRD_VIN: no longer U107.A5, U107.A6, U107.A7, U107.A8
- net Chainbus.RX: now also R117.2, U101.2 (DATA); no longer J105.9 (Pin_9), J108.9 (Pin_9)
- net Chainbus.SCL: now also J104.1 (Pin_1); no longer J104.2 (Pin_2)
- net Chainbus.SDA: now also J102.1 (Pin_1); no longer J102.2 (Pin_2)
- net Chainbus.TX: now also R118.2, U104.1 (INT#)
- net Chainbus_addr0: now also R102.1
- net Chainbus_addr1: now also U102.4 (A3)
- net Chainbus_addr2: now also R128.2, U102.19 (OE#)
- net Chainbus_addr3: now also R104.1, S101.1 (A)
- net Chainbus_addr4: now also R101.1
- net Chainbus_addr5: now also R125.2, R126.1
- net Chainbus_addr6: now also U108.4 (A3)
- net Chainbus_addr7: now also R141.2, U108.19 (OE#)
- net E2_P14: now reaches R135.2, R142.1, S107.1 (A)
- net E2_P14: now also U103.17 (P14); no longer U103.9 (P05)
- net E1_P14: now reaches U104.17 (P14)
- net E1_P14: now also R106.1, R130.2, S102.1 (A)
- net E1_P15: now reaches U104.18 (P15)
- net E1_P15: now also R105.1, R129.1, S103.1 (A)
- net E1_P16: now reaches U104.19 (P16)
- net E1_P16: now also R109.1
- net E1_P17: now reaches U104.20 (P17)
- net E1_P17: now also R110.1
- net at U104.22 (SCL): now also J104.2 (Pin_2); no longer J104.1 (Pin_1)
- net at U104.23 (SDA): now also J102.2 (Pin_2); no longer J102.1 (Pin_1)
- net at U104.5 (P01): no longer R109.1
- net at U104.6 (P02): no longer R110.1
- net E3_P14: now reaches R112.2, R114.1, S105.1 (A)
- net E3_P14: now also U105.17 (P14); no longer U105.7 (P03)
- net E2_P15: now reaches R134.1, R140.1, S106.1 (A)
- net E2_P15: now also U103.18 (P15); no longer U103.8 (P04)
- net at U103.6 (P02): no longer R138.1
- net E2_P16: now reaches U103.19 (P16)
- net E2_P16: now also R137.1
- net E2_P17: now reaches U103.20 (P17)
- net E2_P17: now also R138.1
- net at U103.5 (P01): no longer R137.1
- net E3_P15: now reaches R108.1, R113.1, S104.1 (A)
- net E3_P15: now also U105.18 (P15); no longer U105.6 (P02)
- net at U105.4 (P00): no longer R120.1
- net E3_P16: now reaches U105.19 (P16)
- net E3_P16: now also R120.1
- net E3_P17: now reaches U105.20 (P17)
- net E3_P17: now also R121.1
- net at U105.5 (P01): no longer R121.1
- removed net ECL: J105.10 (Pin_10), J105.6 (Pin_6), J105.8 (Pin_8), J108.10 (Pin_10), J108.6 (Pin_6), J108.8 (Pin_8), R101.1, R102.1, R104.1, R117.2, R118.2, R125.2, R126.1, R128.2, R141.2, R143.2, R144.1, S101.1 (A), U101.2 (DATA), U102.19 (OE#), U102.4 (A3), U104.1 (INT#), U108.19 (OE#), U108.4 (A3)
- now unconnected: U104.8 (P04), U104.9 (P05)
- no-connect marks 55 -> 64
Other:
- note removed: "ALTMODE HEADER"
